Commit message: Update controller parameters and improve Gazebo plugin configuration

File: description/gazebo_control.xacro (robot description, xacro)
@@ -2,5 +2,5 @@
 <robot xmlns:xacro="http://www.ros.org/wiki/xacro">
     <gazebo>
-        <plugin name='diff_drive' filename='libgazebo_ros_diff_drive.so'>
+        <plugin name="gz::sim::systems::DiffDrive" filename="gz-sim-diff-drive-system">
             <!-- Wheel Information -->
             <left_joint>base_left_rear_wheel_joint</left_joint>
@@ -11,12 +11,20 @@
             <wheel_diameter>0.09</wheel_diameter>
             <!-- Limits -->
-            <max_wheel_torque>200</max_wheel_torque>
-            <max_wheel_acceleration>10.0</max_wheel_acceleration>
+            <!-- <max_wheel_torque>200</max_wheel_torque> -->
+            <max_linear_acceleration>0.33</max_linear_acceleration>
+            <!-- Input -->
+            <topic>cmd_vel</topic>
             <!-- Output -->
-            <odometry_frame>odom</odometry_frame>
-            <robot_base_frame>base_footprint</robot_base_frame>
-            <publish_odom>true</publish_odom>
-            <publish_odom_tf>true</publish_odom_tf>
-            <publish_wheel_tf>true</publish_wheel_tf>
+            <frame_id>odom</frame_id>
+            <child_frame_id>base_link</child_frame_id>
+            <odom_topic>odom</odom_topic>
+            <odom_publisher_frequency>30</odom_publisher_frequency>
+            <tf_topic>/tf</tf_topic>
+        </plugin>
+        <plugin filename="gz-sim-joint-state-publisher-system"
+            name="gz::sim::systems::JointStatePublisher">
+            <topic>joint_states</topic>
+            <joint_name>left_wheel_joint</joint_name>
+            <joint_name>right_wheel_joint</joint_name>
         </plugin>
     </gazebo>

File: description/guilassas.xacro (robot description, xacro)
@@ -8,5 +8,4 @@
         <color rgba="0.7 0.7 0.7 1"/>
     </material>
-    <link name="base_footprint"/>
     <link name="base_link">
         <visual>
@@ -114,9 +113,4 @@
         </xacro:inertial_cylinder>
     </link>
-    <joint name="base_footprint_joint" type="fixed">
-        <parent link="base_footprint"/>
-        <child link="base_link" />
-        <origin xyz="0 0 0.03" rpy= "0 0 0" />
-    </joint>
     <joint name="base_lidar_joint" type="fixed">
         <parent link="base_link"/>

File: description/robot.urdf.xacro (robot description, xacro)
@@ -2,5 +2,9 @@
 <robot xmlns:xacro="http://www.ros.org/wiki/xacro"  name="robot">
     <xacro:include filename="guilassas.xacro" />
-    <!--xacro:include filename="gazebo_control.xacro"/-->
-    <xacro:include filename="ros2_control.xacro"/>
+    <xacro:if value="$(arg use_ros2_control)">
+        <xacro:include filename="ros2_control.xacro" />
+    </xacro:if>
+    <xacro:unless value="$(arg use_ros2_control)">
+        <xacro:include filename="gazebo_control.xacro" />
+    </xacro:unless>
 </robot>

Commit message: slam

File: description/gazebo_control.xacro (robot description, xacro)
@@ -9,9 +9,9 @@
             <right_joint>base_right_rear_wheel_joint</right_joint>
             <right_joint>base_right_front_wheel_joint</right_joint>
-            <wheel_separation>0.0675</wheel_separation>
+            <wheel_separation>0.135</wheel_separation>
             <wheel_diameter>0.09</wheel_diameter>
             <!-- Limits -->
             <!-- <max_wheel_torque>200</max_wheel_torque> -->
-            <max_linear_acceleration>0.33</max_linear_acceleration>
+            <max_linear_acceleration>200</max_linear_acceleration>
             <!-- Input -->
             <topic>cmd_vel</topic>

File: description/guilassas.xacro (robot description, xacro)
@@ -26,4 +26,10 @@
         </xacro:inertial_box>
     </link>
+    <link name="base_footprint"/>
+    <joint name="base_footprint_joint" type="fixed">
+        <parent link="base_link"/>
+        <child link="base_footprint" />
+        <origin xyz="0 0 -0.035" rpy= "0 0 0" />
+    </joint>
     <link name="left_rear_wheel">
         <visual>

File: description/lidar.xacro (robot description, xacro)
@@ -29,5 +29,5 @@
             <pose> 0 0 0 0 0 0 </pose>
             <visualize>true</visualize>
-            <update_rate>10</update_rate>
+            <update_rate>30</update_rate>
             <lidar>
                 <scan>

File: description/robot.urdf.xacro (robot description, xacro)
@@ -11,3 +11,4 @@
     </xacro:unless>
     <xacro:include filename="lidar.xacro" />
+    <xacro:include filename="camera.xacro" />
 </robot>
