Commit message: Add Lidar configuration in XACRO file for robot description

File: description/guilassas.xacro (robot description, xacro)
@@ -25,19 +25,4 @@
         <origin xyz="0 0 0.05" rpy="0 0 0"/>
         </xacro:inertial_box>
-    </link>
-    <link name="lidar">
-        <visual>
-            <geometry>
-                <cylinder  radius="0.025" length="0.02"/>
-            </geometry>
-            <origin xyz="0 0 0" rpy= "0 0 0" />
-            <material name="grey" />
-        </visual>
-        <collision>
-            <geometry>
-                <cylinder  radius="0.025" length="0.02"/>
-            </geometry>
-            <origin xyz="0 0 0" rpy= "0 0 0" />
-        </collision>
     </link>
     <link name="left_rear_wheel">
@@ -113,9 +98,4 @@
         </xacro:inertial_cylinder>
     </link>
-    <joint name="base_lidar_joint" type="fixed">
-        <parent link="base_link"/>
-        <child link="lidar" />
-        <origin xyz="0.05 0 0.11" rpy= "0 0 0" />
-    </joint>
     <joint name="base_left_rear_wheel_joint" type="continuous">
         <parent link="base_link"/>

File: description/robot.urdf.xacro (robot description, xacro)
@@ -10,3 +10,4 @@
         <xacro:include filename="gazebo_control.xacro" />
     </xacro:unless>
+    <xacro:include filename="lidar.xacro" />
 </robot>

Commit message: Add URDF and XACRO files for the 'sucata' robot model
- Created robot.xacro to define the robot structure and include necessary files.
- Added ros2_control.xacro for ROS 2 control integration with defined joints and command interfaces.
- Introduced urdf2.csv for defining the robot's physical properties and visual representations.
- Generated urdf2.urdf from SolidWorks, detailing the robot's links, joints, and inertial properties.
- Created urdf2.xacro to provide a structured representation of the robot's components and joints.

File: description/guilassas.xacro (robot description, xacro)
@@ -30,5 +30,5 @@
         <parent link="base_link"/>
         <child link="base_footprint" />
-        <origin xyz="0 0 -0.035" rpy= "0 0 0" />
+        <origin xyz="0 0 0" rpy= "0 0 0" />
     </joint>
     <link name="left_rear_wheel">

File: description/robot.urdf.xacro (robot description, xacro)
@@ -12,3 +12,4 @@
     <xacro:include filename="lidar.xacro" />
     <xacro:include filename="camera.xacro" />
+    <xacro:include filename="imu.xacro" />
 </robot>
