Commit message: Add IMU and ultrasonic sensor models with Gazebo integration
- Created IMU model in urdf/imu.xacro with fixed joint to base_link, including visual, collision, and inertial properties.
- Integrated IMU sensor with Gazebo, specifying sensor parameters and plugin for simulation.
- Added materials definitions in urdf/includes/materials.urdf.xacro for various colors used in models.
- Developed ultrasonic sensor model in urdf/sonar.xacro with fixed joint to base_link, including visual representation and Gazebo sensor configuration.

File: urdf/lidar.xacro (robot description, xacro)
@@ -60,16 +60,16 @@
             <pose> 0 0 0.06 0 0 0 </pose>
             <visualize>true</visualize>
-            <update_rate>30</update_rate>
+            <update_rate>10</update_rate>
             <lidar>
                 <scan>
                     <horizontal>
-                        <samples>360</samples>
-                        <min_angle>-3.14</min_angle>
-                        <max_angle>3.14</max_angle>
+                        <samples>682</samples>
+                        <min_angle>-2.094</min_angle>
+                        <max_angle>2.094</max_angle>
                     </horizontal>
                 </scan>
                 <range>
-                    <min>0.3</min>
-                    <max>12</max>
+                    <min>0.06</min>
+                    <max>4.0</max>
                 </range>
             </lidar>

File: urdf/robot.xacro (robot description, xacro)
@@ -6,3 +6,4 @@
     <xacro:include filename="ros2_control.xacro" />
     <xacro:include filename="lidar.xacro" />
+    <xacro:include filename="imu.xacro" />
 </robot>

File: urdf/urdf2.xacro (robot description, xacro)
@@ -1,156 +1,289 @@
 <?xml version="1.0" encoding="utf-8"?>
-<robot xmlns:xacro="http://ros.org/wiki/xacro" name="sucata">
-  <!-- Base link -->
-  <link name="base_link">
-    <inertial>
-      <origin xyz="0.0014564 0.00032017 0.02708" rpy="0 0 0" />
-      <mass value="0.29402" />
-      <inertia ixx="0.00054056" ixy="-1.0152E-08" ixz="6.2563E-09"
-               iyy="0.0012531" iyz="1.8536E-10" izz="0.0017493" />
-    </inertial>
-    <visual>
-      <origin xyz="0 0 0" rpy="0 0 0" />
-      <geometry>
-        <mesh filename="package://sucata/meshes/base_link.STL" />
-      </geometry>
-      <material name="verde_claro">
-        <color rgba="0.5 1.0 0.5 1"/>
-      </material>
-    </visual>
-    <collision>
-      <origin xyz="0 0 0" rpy="0 0 0" />
-      <geometry>
-        <mesh filename="package://sucata/meshes/base_link.STL" />
-      </geometry>
-    </collision>
-  </link>
-  <!-- Roda FE -->
-  <link name="rodaFE">
-    <inertial>
-      <origin xyz="4.33708624569817E-13 -0.0116000427495452 3.641063145432E-13" rpy="0 0 0" />
-      <mass value="0.0417534418555908" />
-      <inertia ixx="2.90386422409949E-05" ixy="-9.63351560872344E-17" ixz="-1.16755116343788E-16"
-               iyy="4.53732000489224E-05" iyz="-1.07562778637676E-16" izz="2.90386422317585E-05" />
-    </inertial>
-    <visual>
-      <origin xyz="0 0 0" rpy="0 0 0" />
-      <geometry>
-        <mesh filename="package://sucata/meshes/rodaFE.STL" />
-      </geometry>
-      <material name="preto">
-        <color rgba="0.1 0.1 0.1 1"/>
-      </material>
-    </visual>
-    <collision>
-      <origin xyz="0 0 0" rpy="0 0 0" />
-      <geometry>
-        <mesh filename="package://sucata/meshes/rodaFE.STL" />
-      </geometry>
-    </collision>
-  </link>
-  <!-- Roda TE -->
-  <link name="rodaTE">
-    <inertial>
-      <origin xyz="4.33729441251529E-13 -0.0116000427495452 3.64085497861488E-13" rpy="0 0 0" />
-      <mass value="0.0417534418555908" />
-      <inertia ixx="2.90386422409949E-05" ixy="-9.63357589960055E-17" ixz="-1.1675601730821E-16"
-               iyy="4.53732000489224E-05" iyz="-1.07560295850229E-16" izz="2.90386422317585E-05" />
-    </inertial>
-    <visual>
-      <origin xyz="0 0 0" rpy="0 0 0" />
-      <geometry>
-        <mesh filename="package://sucata/meshes/rodaTE.STL" />
-      </geometry>
-      <material name="preto">
-        <color rgba="0.1 0.1 0.1 1"/>
-      </material>
-    </visual>
-    <collision>
-      <origin xyz="0 0 0" rpy="0 0 0" />
-      <geometry>
-        <mesh filename="package://sucata/meshes/rodaTE.STL" />
-      </geometry>
-    </collision>
-  </link>
-  <!-- Roda FD -->
-  <link name="rodaFD">
-    <inertial>
-      <origin xyz="-4.33708624569817E-13 0.0116000427495451 3.64003965858117E-13" rpy="0 0 0" />
-      <mass value="0.0417534418555909" />
-      <inertia ixx="2.90386422409949E-05" ixy="-9.63348726903862E-17" ixz="1.16761894791001E-16"
-               iyy="4.53732000489225E-05" iyz="1.07446973492785E-16" izz="2.90386422317586E-05" />
-    </inertial>
-    <visual>
-      <origin xyz="0 0 0" rpy="0 0 0" />
-      <geometry>
-        <mesh filename="package://sucata/meshes/rodaFD.STL" />
-      </geometry>
-      <material name="preto">
-        <color rgba="0.1 0.1 0.1 1"/>
-      </material>
-    </visual>
-    <collision>
-      <origin xyz="0 0 0" rpy="0 0 0" />
-      <geometry>
-        <mesh filename="package://sucata/meshes/rodaFD.STL" />
-      </geometry>
-    </collision>
-  </link>
-  <!-- Roda TD -->
-  <link name="rodaTD">
-    <inertial>
-      <origin xyz="-4.33729441251529E-13 0.0116000427495451 3.64019578369401E-13" rpy="0 0 0" />
-      <mass value="0.0417534418555909" />
-      <inertia ixx="2.9038642240995E-05" ixy="-9.63350567825533E-17" ixz="1.16754828991177E-16"
-               iyy="4.53732000489225E-05" iyz="1.07446496399349E-16" izz="2.90386422317586E-05" />
-    </inertial>
-    <visual>
-      <origin xyz="0 0 0" rpy="0 0 0" />
-      <geometry>
-        <mesh filename="package://sucata/meshes/rodaTD.STL" />
-      </geometry>
-      <material name="preto">
-        <color rgba="0.1 0.1 0.1 1"/>
-      </material>
-    </visual>
-    <collision>
-      <origin xyz="0 0 0" rpy="0 0 0" />
-      <geometry>
-        <mesh filename="package://sucata/meshes/rodaTD.STL" />
-      </geometry>
-    </collision>
-  </link>
-  <!-- Joints -->
-  <joint name="roda_FE" type="continuous">
-    <origin xyz="0.0815 0.0973 0.0115" rpy="0 0 0" />
-    <parent link="base_link" />
-    <child link="rodaFE" />
-    <axis xyz="0 1 0" />
-    <limit effort="10" velocity="10" />
-    <dynamics damping="0.1" friction="0.1" />
-  </joint>
-  <joint name="roda_TE" type="continuous">
-    <origin xyz="-0.0815 0.0973 0.0115" rpy="0 0 0" />
-    <parent link="base_link" />
-    <child link="rodaTE" />
-    <axis xyz="0 1 0" />
-    <limit effort="10" velocity="10" />
-    <dynamics damping="0.1" friction="0.1" />
-  </joint>
-  <joint name="roda_FD" type="continuous">
-    <origin xyz="0.0814999999999993 -0.0973000000000006 0.0115000000000003" rpy="0 0 0" />
-    <parent link="base_link" />
-    <child link="rodaFD" />
-    <axis xyz="0 1 0" />
-    <limit effort="10" velocity="10" />
-    <dynamics damping="0.1" friction="0.1" />
-  </joint>
-  <joint name="roda_TD" type="continuous">
-    <origin xyz="-0.0815 -0.0973 0.0115" rpy="0 0 0" />
-    <parent link="base_link" />
-    <child link="rodaTD" />
-    <axis xyz="0 1 0" />
-    <limit effort="10" velocity="10" />
-    <dynamics damping="0.1" friction="0.1" />
+<!-- This URDF was automatically created by SolidWorks to URDF Exporter! Originally created by Stephen Brawner (brawner@gmail.com)
+     Commit Version: 1.6.0-4-g7f85cfe  Build Version: 1.6.7995.38578
+     For more information, please see http://wiki.ros.org/sw_urdf_exporter -->
+<robot
+  name="sucata">
+  <link name="base_footprint"/>
+    <joint name="base_footprint_joint" type="fixed">
+        <parent link="base_link"/>
+        <child link="base_footprint" />
+        <origin xyz="0.0014564 0.00032017 -0.029" rpy="0 0 0" />
+    </joint>
+  <link
+    name="base_link">
+    <inertial>
+      <origin
+        xyz="0.0014564 0.00032017 0.02708"
+        rpy="0 0 0" />
+      <mass
+        value="0.29402" />
+      <inertia
+        ixx="0.00054056"
+        ixy="-1.0152E-08"
+        ixz="6.2563E-09"
+        iyy="0.0012531"
+        iyz="1.8536E-10"
+        izz="0.0017493" />
+    </inertial>
+    <visual>
+      <origin
+        xyz="0 0 0"
+        rpy="0 0 0" />
+      <geometry>
+        <mesh
+          filename="package://sucata/meshes/base_link.STL" />
+      </geometry>
+      <material
+        name="verde_claro">
+        <color
+          rgba="0.5 1.0 0.5 1"/>
+      </material>
+    </visual>
+    <collision>
+      <origin
+        xyz="0 0 0"
+        rpy="0 0 0" />
+      <geometry>
+        <mesh
+          filename="package://sucata/meshes/base_link.STL" />
+      </geometry>
+    </collision>
+  </link>
+  <link
+    name="rodaFE">
+    <inertial>
+      <origin
+        xyz="4.33708624569817E-13 -0.0116000427495452 3.641063145432E-13"
+        rpy="0 0 0" />
+      <mass
+        value="0.0417534418555908" />
+      <inertia
+        ixx="2.90386422409949E-05"
+        ixy="-9.63351560872344E-17"
+        ixz="-1.16755116343788E-16"
+        iyy="4.53732000489224E-05"
+        iyz="-1.07562778637676E-16"
+        izz="2.90386422317585E-05" />
+    </inertial>
+    <visual>
+      <origin
+        xyz="0 0 0"
+        rpy="0 0 0" />
+      <geometry>
+        <mesh
+          filename="package://sucata/meshes/rodaFE.STL" />
+      </geometry>
+      <material
+        name="preto">
+        <color
+          rgba="0.1 0.1 0.1 1"/>
+      </material>
+    </visual>
+    <collision>
+      <origin
+        xyz="0 0 0"
+        rpy="0 0 0" />
+      <geometry>
+        <mesh
+          filename="package://sucata/meshes/rodaFE.STL" />
+      </geometry>
+    </collision>
+  </link>
+  <joint
+    name="roda_FE"
+    type="continuous">
+    <origin
+      xyz="0.0815 0.0973 0.0115"
+      rpy="0 0 0" />
+    <parent
+      link="base_link" />
+    <child
+      link="rodaFE" />
+    <axis
+      xyz="0 1 0" />
+    <limit
+      effort="10"
+      velocity="10" />
+    <dynamics
+      damping="0.1"
+      friction="0.1" />
+  </joint>
+  <link
+    name="rodaTE">
+    <inertial>
+      <origin
+        xyz="4.33729441251529E-13 -0.0116000427495452 3.64085497861488E-13"
+        rpy="0 0 0" />
+      <mass
+        value="0.0417534418555908" />
+      <inertia
+        ixx="2.90386422409949E-05"
+        ixy="-9.63357589960055E-17"
+        ixz="-1.1675601730821E-16"
+        iyy="4.53732000489224E-05"
+        iyz="-1.07560295850229E-16"
+        izz="2.90386422317585E-05" />
+    </inertial>
+    <visual>
+      <origin
+        xyz="0 0 0"
+        rpy="0 0 0" />
+      <geometry>
+        <mesh
+          filename="package://sucata/meshes/rodaTE.STL" />
+      </geometry>
+      <material
+        name="preto">
+        <color
+          rgba="0.1 0.1 0.1 1"/>
+      </material>
+    </visual>
+    <collision>
+      <origin
+        xyz="0 0 0"
+        rpy="0 0 0" />
+      <geometry>
+        <mesh
+          filename="package://sucata/meshes/rodaTE.STL" />
+      </geometry>
+    </collision>
+  </link>
+  <joint
+    name="roda_TE"
+    type="continuous">
+    <origin
+      xyz="-0.0815 0.0973 0.0115"
+      rpy="0 0 0" />
+    <parent
+      link="base_link" />
+    <child
+      link="rodaTE" />
+    <axis
+      xyz="0 1 0" />
+    <limit
+      effort="10"
+      velocity="10" />
+    <dynamics
+      damping="0.1"
+      friction="0.1" />
+  </joint>
+  <link
+    name="rodaFD">
+    <inertial>
+      <origin
+        xyz="-4.33708624569817E-13 0.0116000427495451 3.64003965858117E-13"
+        rpy="0 0 0" />
+      <mass
+        value="0.0417534418555909" />
+      <inertia
+        ixx="2.90386422409949E-05"
+        ixy="-9.63348726903862E-17"
+        ixz="1.16761894791001E-16"
+        iyy="4.53732000489225E-05"
+        iyz="1.07446973492785E-16"
+        izz="2.90386422317586E-05" />
+    </inertial>
+    <visual>
+      <origin
+        xyz="0 0 0"
+        rpy="0 0 0" />
+      <geometry>
+        <mesh
+          filename="package://sucata/meshes/rodaFD.STL" />
+      </geometry>
+      <material
+        name="preto">
+        <color
+          rgba="0.1 0.1 0.1 1"/>
+      </material>
+    </visual>
+    <collision>
+      <origin
+        xyz="0 0 0"
+        rpy="0 0 0" />
+      <geometry>
+        <mesh
+          filename="package://sucata/meshes/rodaFD.STL" />
+      </geometry>
+    </collision>
+  </link>
+  <joint
+    name="roda_FD"
+    type="continuous">
+    <origin
+      xyz="0.0814999999999993 -0.0973000000000006 0.0115000000000003"
+      rpy="0 0 0" />
+    <parent
+      link="base_link" />
+    <child
+      link="rodaFD" />
+    <axis
+      xyz="0 1 0" />
+    <limit
+      effort="10"
+      velocity="10" />
+    <dynamics
+      damping="0.1"
+      friction="0.1" />
+  </joint>
+  <link
+    name="rodaTD">
+    <inertial>
+      <origin
+        xyz="-4.33729441251529E-13 0.0116000427495451 3.64019578369401E-13"
+        rpy="0 0 0" />
+      <mass
+        value="0.0417534418555909" />
+      <inertia
+        ixx="2.9038642240995E-05"
+        ixy="-9.63350567825533E-17"
+        ixz="1.16754828991177E-16"
+        iyy="4.53732000489225E-05"
+        iyz="1.07446496399349E-16"
+        izz="2.90386422317586E-05" />
+    </inertial>
+    <visual>
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