Commit message: Update configuration files for improved robot simulation and sensor integration
- Change base frame ID from 'base_link' to 'base_footprint' in amcl.yaml and ekf.yaml
- Update IMU and LIDAR sensor parameters in respective XACRO files
- Modify launch file to include gazebo parameters
- Adjust mapping parameters in mapper_params_online_async.yaml
- Add gazebo_params.yaml for simulation settings
- Refactor joint definitions in urdf files for better structure

File: urdf/imu.xacro (robot description, xacro)
@@ -44,5 +44,5 @@
         <sensor name="imu_sensor" type="imu">
             <always_on>1</always_on>
-            <update_rate>50</update_rate>
+            <update_rate>100</update_rate>
             <visualize>true</visualize>
             <topic>imu</topic>
@@ -50,4 +50,5 @@
                 name="gz::sim::systems::Imu">
             </plugin>
+            <gz_frame_id>lidar</gz_frame_id>
         </sensor>
     </gazebo>

File: urdf/lidar.xacro (robot description, xacro)
@@ -60,5 +60,5 @@
             <pose> 0 0 0.06 0 0 0 </pose>
             <visualize>true</visualize>
-            <update_rate>10</update_rate>
+            <update_rate>30</update_rate>
             <lidar>
                 <scan>

File: urdf/urdf2.xacro (robot description, xacro)
@@ -6,8 +6,8 @@
   name="sucata">
   <link name="base_footprint"/>
-    <joint name="base_footprint_joint" type="fixed">
-        <parent link="base_link"/>
-        <child link="base_footprint" />
-        <origin xyz="0.0014564 0.00032017 -0.029" rpy="0 0 0" />
+    <joint name="base_joint" type="fixed">
+        <parent link="base_footprint"/>
+        <child link="base_link" />
+        <origin xyz="0.0014564 0.00032017 0.05608" rpy="0 0 0" />
     </joint>
   <link

Commit message: Add URDF definition for camera with depth sensor integration
- Created a new URDF file for the camera, including its link and joint definitions.
- Defined inertial properties, visual and collision geometries for the camera link.
- Added a fixed joint connecting the camera to the base link.
- Integrated a depth sensor configuration for use with ROS 2 and Gazebo, specifying camera parameters such as field of view, image resolution, and clipping distances.

File: urdf/imu.xacro (robot description, xacro)
@@ -1,14 +1,20 @@
 <?xml version="1.0"?>
 <robot xmlns:xacro="http://www.ros.org/wiki/xacro" >
-    <joint name="imu_joint" type="fixed">
-    <origin
-      xyz="0.063662 0.0019005 0.0585"
-      rpy="0 0 0" />
-    <parent
-      link="base_link" />
-    <child
-      link="imu" />
-  </joint>
-    <link name="imu">
+    <link
+    name="imu">
+    <inertial>
+      <origin
+        xyz="1.58927283510988E-05 9.32559180236298E-05 0.000878239070510656"
+        rpy="0 0 0" />
+      <mass
+        value="0.000641531141315228" />
+      <inertia
+        ixx="3.17041200198106E-08"
+        ixy="1.24863172344468E-11"
+        ixz="-4.01457310722804E-14"
+        iyy="1.18309245142538E-08"
+        iyz="-1.71325876343045E-15"
+        izz="4.3260264266368E-08" />
+    </inertial>
     <visual>
       <origin
@@ -22,5 +28,5 @@
         name="">
         <color
-          rgba="0.17647 0.2902 0.8 1" />
+          rgba="0.176470588235294 0.290196078431373 0.8 1" />
       </material>
     </visual>
@@ -34,10 +40,18 @@
       </geometry>
     </collision>
-    <inertial>
-            <mass value="0.1"/>
-            <origin xyz="0 0 0" rpy="0 0 0"/>
-            <inertia ixx="0.001" ixy="0" ixz="0" iyy="0.001" iyz="0" izz="0.001"/>
-    </inertial>
   </link>
+  <joint
+    name="imu_joint"
+    type="fixed">
+    <origin
+      xyz="-0.034597 0 0.09"
+      rpy="0 0 0" />
+    <parent
+      link="base_link" />
+    <child
+      link="imu" />
+    <axis
+      xyz="0 0 0" />
+  </joint>
     <gazebo reference="imu">
         <material>Gazebo/Red</material>

File: urdf/robot.xacro (robot description, xacro)
@@ -7,3 +7,4 @@
     <xacro:include filename="lidar.xacro" />
     <xacro:include filename="imu.xacro" />
+    <xacro:include filename="camera.xacro" />
 </robot>
