Commit message: points

File: urdf/camera.xacro (robot description, xacro)
@@ -56,25 +56,25 @@
   </joint>
   <!-- Sensor para ROS 2 + Gazebo -->
-  <gazebo reference="camera_link">
-    <material>Gazebo/Red</material>
-    <sensor name="camera" type="depth">
-      <pose>0 0 0 0 0 0</pose>
-      <visualize>true</visualize>
-      <update_rate>10</update_rate>
-      <camera>
-        <horizontal_fov>1.089</horizontal_fov>
-        <image>
-          <width>640</width>
-          <height>480</height>
-          <format>R8G8B8</format>
-        </image>
-        <clip>
-          <near>0.05</near>
-          <far>8.0</far>
-        </clip>
-      </camera>
-      <!-- <topic>camera/image_raw</topic> -->
-      <gz_frame_id>camera_link_optical</gz_frame_id>
-    </sensor>
-  </gazebo>
+    <gazebo reference="camera_link">
+        <material>Gazebo/Red</material>
+        <sensor name="camera" type="depth">
+            <pose> 0 0 0 0 0 0 </pose>
+            <visualize>true</visualize>
+            <update_rate>30</update_rate>
+            <camera>
+                <horizontal_fov>1.089</horizontal_fov>
+                <image>
+                    <format>B8G8R8</format>
+                    <width>640</width>
+                    <height>480</height>
+                </image>
+                <clip>
+                    <near>0.05</near>
+                    <far>8.0</far>
+                </clip>
+            </camera>
+            <topic>/world/mundoArUco/model/sucata/link/base_footprint/sensor/camera/depth_image</topic>
+            <gz_frame_id>camera_link</gz_frame_id>
+        </sensor>
+    </gazebo>
 </robot>

Commit message: ajustes finais e fotos

File: urdf/camera.xacro (robot description, xacro)
@@ -56,9 +56,9 @@
   </joint>
     <gazebo reference="camera_link">
-        <material>Gazebo/Red</material>
+        <material>Gazebo/Grey</material>
         <sensor name="cameraV3" type="camera">
             <pose> 0 0 0 0 0 0 </pose>
             <visualize>true</visualize>
-            <update_rate>10</update_rate>
+            <update_rate>60</update_rate>
             <camera>
                 <horizontal_fov>1.089</horizontal_fov>

File: urdf/depthCamera.xacro (robot description, xacro)
@@ -55,5 +55,5 @@
   </joint>
   <gazebo reference="depth_link">
-    <material>Gazebo/Red</material>
+    <material>Gazebo/Grey</material>
     <sensor name="xtion_depth" type="depth">
       <pose>0 0 0 0 0 0</pose>
